Commit message: 这是修改执行器可插拔架构前的较完善版本

File: src/uuv_description/urdf/lauv_model.xacro (robot description, xacro)
@@ -45,5 +45,5 @@
       <origin xyz="${x} ${y} ${z}" rpy="${r} ${p} ${yaw}"/>
       <axis xyz="0 0 1"/>
-      <limit lower="-0.785" upper="0.785" effort="10" velocity="10"/>
+      <limit lower="-0.5237" upper="0.5237" effort="10" velocity="10"/>
     </joint>
   </xacro:macro>

Commit message: 20260228晚上: 完成了集群化的前两步,nodelet机制已经搭建完毕,下一步是建立uuv_director,自动通过nodelet自动载入UUV集群到场景中,而不需要launch文件

File: src/uuv_description/urdf/lauv_model.xacro (robot description, xacro)
@@ -14,5 +14,5 @@
   <xacro:include filename="$(find uuv_description)/urdf/plugins/guidances/to_goal_guidance.xacro" />
   <xacro:if value="${'$(arg dynamics_type)' == 'fossen'}">
-      <xacro:insert_fossen_dynamics update_rate="100.0" />
+      <xacro:insert_fossen_dynamics update_rate="100.0" is_pub_actuator_state="false" />
   </xacro:if>
   <xacro:if value="${'$(arg dynamics_type)' == 'first_order'}">

File: src/uuv_description/urdf/plugins/actuators/lauv_actuator.xacro (robot description, xacro)
@@ -1,5 +1,5 @@
 <?xml version="1.0"?>
 <robot xmlns:xacro="http://www.ros.org/wiki/xacro">
-    <xacro:macro name="insert_lauv_actuator">
+    <xacro:macro name="insert_lauv_actuator" >
         <plugin layer="actuator" name="lauv_actuator" type="uuv_control/LauvActuator">
             <thruster>

File: src/uuv_description/urdf/plugins/dynamics/lauv_fossen_dynamics.xacro (robot description, xacro)
@@ -1,5 +1,5 @@
 <?xml version="1.0"?>
 <robot xmlns:xacro="http://www.ros.org/wiki/xacro">
-    <xacro:macro name="insert_fossen_dynamics" params="update_rate:=100.0">
+    <xacro:macro name="insert_fossen_dynamics" params="update_rate:=100.0 is_pub_actuator_state:=false">
         <plugin layer="dynamics" name="fossen_model" type="uuv_control/FossenDynamics">
             <update_rate>${update_rate}</update_rate>
@@ -10,4 +10,5 @@
             <neutrally_buoyant>true</neutrally_buoyant>
             <publish_debug_visuals>true</publish_debug_visuals>
+            <is_pub_actuator_state>${is_pub_actuator_state}</is_pub_actuator_state>
             <cog>0.0 0.0 0.0</cog>
             <cob>0.0 0.0 -0.01</cob>

Commit message: 20260301晚_已经将当前的各层控制架构优化完毕,并且测试目前的各项功能均正常,下一步工作,1_添加碰撞检测话题的发布,2_实现Flocking+改进APF的Guidance算法git add .!

File: src/uuv_description/urdf/lauv_model.xacro (robot description, xacro)
@@ -2,29 +2,25 @@
 <robot name="lauv" xmlns:xacro="http://www.ros.org/wiki/xacro">
   <xacro:arg name="namespace" default="uuv_0"/>
+  <xacro:arg name="dynamics_type" default="fossen" />
+  <xacro:arg name="actuator_type" default="lauv" />
   <xacro:arg name="controller_type" default="pid" />
-  <xacro:arg name="dynamics_type" default="fossen" />
   <xacro:arg name="guidance_type" default="to_goal" />
   <xacro:property name="ns" value="$(arg namespace)"/>
   <xacro:include filename="$(find uuv_description)/urdf/plugins/actuators/lauv_actuator.xacro" />
   <xacro:include filename="$(find uuv_description)/urdf/plugins/dynamics/lauv_fossen_dynamics.xacro" />
-  <xacro:include filename="$(find uuv_description)/urdf/plugins/dynamics/first_order_dynamics.xacro" />
   <xacro:include filename="$(find uuv_description)/urdf/plugins/controllers/pid_controller.xacro" />
-  <xacro:include filename="$(find uuv_description)/urdf/plugins/controllers/teleop_joy_controller.xacro" />
   <xacro:include filename="$(find uuv_description)/urdf/plugins/sensors/simple_2d_sonar.xacro" />
   <xacro:include filename="$(find uuv_description)/urdf/plugins/guidances/to_goal_guidance.xacro" />
   <xacro:if value="${'$(arg dynamics_type)' == 'fossen'}">
-      <xacro:insert_fossen_dynamics update_rate="100.0" is_pub_actuator_state="false" />
+      <xacro:insert_fossen_dynamics update_rate="100.0" publish_debug="true" publish_debug_rate="10.0" />
   </xacro:if>
-  <xacro:if value="${'$(arg dynamics_type)' == 'first_order'}">
-      <xacro:insert_first_order_dynamics update_rate="100.0" />
-  </xacro:if>
+  <xacro:if value="${'$(arg actuator_type)' == 'lauv'}">
+      <xacro:insert_lauv_actuator update_rate="200.0" publish_debug="true" publish_debug_rate="10.0" />
+  </xacro:if>  <!-- 将actuator的更新频率设置的很大，相当于就没有了频率控制，就是调用就触发！ -->
   <xacro:if value="${'$(arg controller_type)' == 'pid'}">
-      <xacro:insert_pid_controller update_rate="10.0" enable_dyn="false" use_local_cmd="true" />
-  </xacro:if>
-  <xacro:if value="${'$(arg controller_type)' == 'teleop'}">
-      <xacro:insert_teleop_controller update_rate="10.0" />
+      <xacro:insert_pid_controller update_rate="10.0" publish_debug="true" publish_debug_rate="10.0" enable_dyn="false" />
   </xacro:if>
   <xacro:if value="${'$(arg guidance_type)' == 'to_goal'}">
-      <xacro:insert_to_goal_guidance update_rate="10.0" use_local_tp="false" cruise_speed="7" acceptance_radius="4.0" max_pitch_deg="40.0" />
+      <xacro:insert_to_goal_guidance update_rate="10.0" publish_debug="true" publish_debug_rate="10.0" cruise_speed="7" acceptance_radius="4.0" max_pitch_deg="40.0" />
   </xacro:if>
   <xacro:insert_simple_2d_sonar name="forward_looking_sonar" update_rate="10.0" beams="30" fov="150.0" max_range="200.0" />

File: src/uuv_description/urdf/plugins/actuators/lauv_actuator.xacro (robot description, xacro)
@@ -1,6 +1,11 @@
 <?xml version="1.0"?>
 <robot xmlns:xacro="http://www.ros.org/wiki/xacro">
-    <xacro:macro name="insert_lauv_actuator" >
+    <xacro:macro name="insert_lauv_actuator"  params="update_rate:=100.0 publish_debug:=true publish_debug_rate:=5.0">
         <plugin layer="actuator" name="lauv_actuator" type="uuv_control/LauvActuator">
+            <!-- ControlPluginBase的参数 -->
+            <update_rate>${update_rate}</update_rate>
+            <publish_debug>${publish_debug}</publish_debug>
+            <publish_debug_rate>${publish_debug_rate}</publish_debug_rate>
+            <!-- LauvActuator 特有的参数 -->
             <thruster>
                 <rotor_constant>0.0002</rotor_constant>

File: src/uuv_description/urdf/plugins/controllers/pid_controller.xacro (robot description, xacro)
@@ -1,9 +1,12 @@
 <?xml version="1.0"?>
 <robot xmlns:xacro="http://www.ros.org/wiki/xacro">
-    <xacro:macro name="insert_pid_controller" params="update_rate:=10.0 enable_dyn:=false use_local_cmd:=false">
+    <xacro:macro name="insert_pid_controller" params="update_rate:=100.0 publish_debug:=true publish_debug_rate:=5.0 enable_dyn:=false">
         <plugin layer="controller" name="pid_ctrl" type="uuv_control/PidController">
+            <!-- ControlPluginBase的参数 -->
             <update_rate>${update_rate}</update_rate>
+            <publish_debug>${publish_debug}</publish_debug>
+            <publish_debug_rate>${publish_debug_rate}</publish_debug_rate>
+            <!--  PidController 特有的参数  -->
             <enable_dynamic_reconfigure>${enable_dyn}</enable_dynamic_reconfigure>
-            <use_local_cmd>${use_local_cmd}</use_local_cmd>
             <kp_u>40.0</kp_u> <ki_u>17.0</ki_u> <kd_u>5.0</kd_u> <max_output_u>200.0</max_output_u> <max_integral_u>50.0</max_integral_u>
             <kp_pitch>0.4</kp_pitch> <ki_pitch>0.0</ki_pitch> <kd_pitch>0.0</kd_pitch> <max_output_pitch>0.8</max_output_pitch> <max_integral_pitch>0.0</max_integral_pitch>

File: src/uuv_description/urdf/plugins/dynamics/lauv_fossen_dynamics.xacro (robot description, xacro)
@@ -1,7 +1,11 @@
 <?xml version="1.0"?>
 <robot xmlns:xacro="http://www.ros.org/wiki/xacro">
-    <xacro:macro name="insert_fossen_dynamics" params="update_rate:=100.0 is_pub_actuator_state:=false">
+    <xacro:macro name="insert_fossen_dynamics" params="update_rate:=100.0 publish_debug:=true publish_debug_rate:=5.0">
         <plugin layer="dynamics" name="fossen_model" type="uuv_control/FossenDynamics">
+            <!-- ControlPluginBase的参数 -->
             <update_rate>${update_rate}</update_rate>
+            <publish_debug>${publish_debug}</publish_debug>
+            <publish_debug_rate>${publish_debug_rate}</publish_debug_rate>
+            <!-- FossenDynamics 特有的参数 -->
             <mass>18.0</mass>
             <volume>0.01755137</volume>
@@ -9,6 +13,4 @@
             <gravity>9.81</gravity>
             <neutrally_buoyant>true</neutrally_buoyant>
-            <publish_debug_visuals>true</publish_debug_visuals>
-            <is_pub_actuator_state>${is_pub_actuator_state}</is_pub_actuator_state>
             <cog>0.0 0.0 0.0</cog>
             <cob>0.0 0.0 -0.01</cob>

File: src/uuv_description/urdf/plugins/guidances/to_goal_guidance.xacro (robot description, xacro)
@@ -1,8 +1,11 @@
 <?xml version="1.0"?>
 <robot xmlns:xacro="http://www.ros.org/wiki/xacro">
-    <xacro:macro name="insert_to_goal_guidance" params="update_rate:=10.0 use_local_tp:=false cruise_speed:=7.7 acceptance_radius:=2.0 max_pitch_deg:=30.0">
+    <xacro:macro name="insert_to_goal_guidance" params="update_rate:=100.0 publish_debug:=true publish_debug_rate:=5.0 cruise_speed:=7.7 acceptance_radius:=2.0 max_pitch_deg:=30.0">
         <plugin layer="guidance" name="to_goal_guidance" type="uuv_control/ToGoalGuidance">
+            <!-- ControlPluginBase的参数 -->
             <update_rate>${update_rate}</update_rate>
-            <use_local_targetpoint_>${use_local_tp}</use_local_targetpoint_>
+            <publish_debug>${publish_debug}</publish_debug>
+            <publish_debug_rate>${publish_debug_rate}</publish_debug_rate>
+            <!-- ToGoalGuidance 特有的参数 -->
             <cruise_speed>${cruise_speed}</cruise_speed>
             <acceptance_radius>${acceptance_radius}</acceptance_radius>

Commit message: 20260302下午_在上一个版本的基础上,将碰撞检测从简单的距离阈值检测升级为了SAT碰撞盒检测,但是还没有在障碍物有旋转角时验证其有效性

File: src/uuv_description/urdf/lauv_model.xacro (robot description, xacro)
@@ -32,9 +32,15 @@
       </geometry>
     </visual>
-    <collision>
+    <!-- <collision>
       <origin xyz="0 0 0" rpy="0 0 0"/>
       <geometry>
         <mesh filename="package://uuv_description/meshes/body.stl"/>
       </geometry>
+    </collision> -->
+    <collision>
+        <origin xyz="0 0 0" rpy="0 1.570796 0" />
+        <geometry>
+            <cylinder length="1.1" radius="0.075" />
+        </geometry>
     </collision>
   </link>
