Commit message: 新增了多连续目标导航的剧本,现在spacialFlockingGuidance已经较为完善了,现在在完成CBBADecision,但是现在需要将neighbors消息的订阅移到ControlNodelet中去,以避免Decision层重复订阅

File: src/uuv_description/urdf/plugins/dynamics/lauv_fossen_dynamics.xacro (robot description, xacro)
@@ -56,5 +56,4 @@
                 0.0  0.0   0.0  0.0   0.0   0.0
             </linear_damping_forward_speed>
-            <xacro:insert_lauv_actuator />
         </plugin>
     </xacro:macro>

File: src/uuv_description/urdf/plugins/guidances/spacial_flocking_guidance.xacro (robot description, xacro)
@@ -50,8 +50,11 @@
             <zeta_n>${zeta_n}</zeta_n>
             <delta_n>${delta_n}</delta_n>
-            <max_ftotal>${k_pull}</max_ftotal>
+            <k_pull>${k_pull}</k_pull>
+            <r_comm>${r_comm}</r_comm>
+            <k_pull>${k_pull}</k_pull>
             <t_ftotal>${r_comm}</t_ftotal>
             <force_lp_gain>${force_lp_gain}</force_lp_gain>
             <flock_force_limit>${flock_force_limit}</flock_force_limit>
+            <!-- 避障力部分 -->
             <d_sense>${d_sense}</d_sense>
             <d_inflation>${d_inflation}</d_inflation>

File: src/uuv_description/urdf/plugins/sensors/simple_2d_sonar.xacro (robot description, xacro)
@@ -1,5 +1,6 @@
 <?xml version="1.0"?>
 <robot xmlns:xacro="http://www.ros.org/wiki/xacro">
-    <xacro:macro name="insert_simple_2d_sonar" params="name:='sonar_front' update_rate:=10.0 beams:=30 fov:=150.0 max_range:=200.0">
+    <xacro:macro name="insert_simple_2d_sonar"
+    params="name:='sonar_front' update_rate:=10.0 beams:=30 fov:=150.0 max_range:=200.0">
         <plugin layer="sensor" name="${name}" type="uuv_sensor/Simple2DSonar">
             <update_rate>${update_rate}</update_rate>
